File: design_files/AST1002.sch (EAGLE design)
At the start: 8 parts, among them J1 SM05B, U1 LSM9DS1

Commit message: updates
Parts:
- C1: value 10uF -> 4.7uF; device tinycircuits:AS-ITM-00002 -> tinycircuits:AS-ITM-00088; PARTNO (none) -> AS-ITM-00088; VALUE (none) -> 4.7uF
- J1: device tinycircuits:AS-ITM-00340 -> tinycircuits:AS-ITM-00340EDGE
